Commit message: Final status update for Report

File: include/urdf/fr3_robot.urdf (robot description, URDF)
Before this commit: robot fr3, 19 links, 18 joints
Links:
- added link fr3_link2_offset1
- added link fr3_link2_offset2
- added link fr3_link7_offset1
Joints:
- added joint fr3_link2_offset1_joint: type fixed, parent fr3_link2, child fr3_link2_offset1, origin xyz=0 0 0.1 rpy=0 0 0
- added joint fr3_link2_offset2_joint: type fixed, parent fr3_link2, child fr3_link2_offset2, origin xyz=0 0 -0.1 rpy=0 0 0
- added joint fr3_link7_offset1_joint: type fixed, parent fr3_link7, child fr3_link7_offset1, origin xyz=0 0 -0.03 rpy=0 0 0
